Commit message: Add files via upload

File: al5d/al5d_description/urdf/al5d.xacro (robot description, xacro)
@@ -2,7 +2,183 @@
 <robot name="al5d" xmlns:xacro="http://www.ros.org/wiki/xacro">
 	<xacro:include filename="$(find al5d_description)/urdf/al5d.gazebo" />
-	<link name="assembly_3_1">
-		<collision>
-			<origin xyz="-0.00970271 -0.0434987 0.100418" rpy="0.037808 1.24896 0.180399" />
+	<link name="wrist_1">
+		<collision>
+			<origin xyz="-0.036586 -0.324104 0.087087" rpy="-2.53263 0.00439039 -3.13599" />
+			<geometry>
+				<mesh filename="file://$(find al5d_description)/urdf/al5d/servo.stl"/>
+			</geometry>
+			<material name="servo_material">
+				<color rgba="0.25098 0.25098 0.25098 1.0"/>
+			</material>
+		</collision>
+		<collision>
+			<origin xyz="-0.036561 -0.325276 0.0854659" rpy="0.608966 0.00439039 -3.13599" />
+			<geometry>
+				<mesh filename="file://$(find al5d_description)/urdf/al5d/part_1.stl"/>
+			</geometry>
+			<material name="part_1_material">
+				<color rgba="0.501961 0.501961 0.501961 1.0"/>
+			</material>
+		</collision>
+		<collision>
+			<origin xyz="-0.0221441 -0.273632 0.146654" rpy="-0.393492 0.00439039 -3.13599" />
+			<geometry>
+				<mesh filename="file://$(find al5d_description)/urdf/al5d/imported15.stl"/>
+			</geometry>
+			<material name="imported15_material">
+				<color rgba="0.917647 0.917647 0.917647 1.0"/>
+			</material>
+		</collision>
+		<collision>
+			<origin xyz="-0.0131671 -0.296957 0.125988" rpy="-2.53263 0.00439039 -3.13599" />
+			<geometry>
+				<mesh filename="file://$(find al5d_description)/urdf/al5d/bb-03.stl"/>
+			</geometry>
+			<material name="bb-03_material">
+				<color rgba="0.647059 0.647059 0.647059 1.0"/>
+			</material>
+		</collision>
+		<collision>
+			<origin xyz="-0.0131671 -0.296957 0.125988" rpy="-0.608966 -0.00439039 0.00560636" />
+			<geometry>
+				<mesh filename="file://$(find al5d_description)/urdf/al5d/imported30.stl"/>
+			</geometry>
+			<material name="imported30_material">
+				<color rgba="0.231373 0.380392 0.705882 1.0"/>
+			</material>
+		</collision>
+		<visual>
+			<origin xyz="0 0 0" rpy="0 -0 0" />
+			<geometry>
+				<mesh filename="file://$(find al5d_description)/urdf/al5d/wrist_1.stl"/>
+			</geometry>
+			<material name="wrist_1_material">
+				<color rgba="0.436028 0.436736 0.438282 1.0"/>
+			</material>
+		</visual>
+		<inertial>
+			<origin xyz="-0.0361093 -0.313655 0.102111" rpy="0 0 0"/>
+			<mass value="0.0622741" />
+			<inertia ixx="2.36538e-05" ixy="-3.8553e-07"  ixz="-7.51646e-07" iyy="4.22717e-05" iyz="-8.54433e-06" izz="3.59672e-05" />
+		</inertial>
+	</link>
+	<link name="elbow_1">
+		<collision>
+			<origin xyz="-0.0244212 -0.0220573 0.0354369" rpy="-1.5708 -0.568339 3.14159" />
+			<geometry>
+				<mesh filename="file://$(find al5d_description)/urdf/al5d/imported11.stl"/>
+			</geometry>
+			<material name="imported11_material">
+				<color rgba="0.231373 0.380392 0.705882 1.0"/>
+			</material>
+		</collision>
+		<collision>
+			<origin xyz="-0.125879 -0.0512165 0.0975185" rpy="-1.5708 -0.568339 3.14159" />
+			<geometry>
+				<mesh filename="file://$(find al5d_description)/urdf/al5d/asb201b.stl"/>
+			</geometry>
+			<material name="asb201b_material">
+				<color rgba="0.498039 0.498039 0.498039 1.0"/>
+			</material>
+		</collision>
+		<collision>
+			<origin xyz="-5.55112e-17 0.0015 5.55112e-17" rpy="-3.95929e-19 7.43601e-17 7.76416e-19" />
+			<geometry>
+				<mesh filename="file://$(find al5d_description)/urdf/al5d/imported8.stl"/>
+			</geometry>
+			<material name="imported8_material">
+				<color rgba="0.231373 0.380392 0.705882 1.0"/>
+			</material>
+		</collision>
+		<collision>
+			<origin xyz="-0.130334 -0.0220573 0.084903" rpy="2.13914 3.52335e-15 1.5708" />
+			<geometry>
+				<mesh filename="file://$(find al5d_description)/urdf/al5d/at-03.stl"/>
+			</geometry>
+			<material name="at-03_material">
+				<color rgba="0.768627 0.886275 0.952941 1.0"/>
+			</material>
+		</collision>
+		<collision>
+			<origin xyz="-0.13301 -0.0220573 0.0866118" rpy="-2.57325 3.57736e-15 1.5708" />
+			<geometry>
+				<mesh filename="file://$(find al5d_description)/urdf/al5d/hub-08.stl"/>
+			</geometry>
+			<material name="hub-08_material">
+				<color rgba="0.917647 0.917647 0.917647 1.0"/>
+			</material>
+		</collision>
+		<collision>
+			<origin xyz="-0.0303533 -0.0379467 0.00732965" rpy="-2.57325 3.4209e-15 1.5708" />
+			<geometry>
+				<mesh filename="file://$(find al5d_description)/urdf/al5d/imported15.stl"/>
+			</geometry>
+			<material name="imported15_material">
+				<color rgba="0.611765 0.811765 0.921569 1.0"/>
+			</material>
+		</collision>
+		<collision>
+			<origin xyz="-0.123429 -0.0220573 0.0986658" rpy="-1.5708 0.568339 -7.43777e-15" />
+			<geometry>
+				<mesh filename="file://$(find al5d_description)/urdf/al5d/imported11.stl"/>
+			</geometry>
+			<material name="imported11_material">
+				<color rgba="0.231373 0.380392 0.705882 1.0"/>
+			</material>
+		</collision>
+		<collision>
+			<origin xyz="0.00113051 -0.0458571 -0.00053094" rpy="1.00246 -3.22359e-15 -1.5708" />
+			<geometry>
+				<mesh filename="file://$(find al5d_description)/urdf/al5d/imported30.stl"/>
+			</geometry>
+			<material name="imported30_material">
+				<color rgba="0.231373 0.380392 0.705882 1.0"/>
+			</material>
+		</collision>
+		<collision>
+			<origin xyz="0.000443529 -0.0274802 0.0168452" rpy="-1.5708 -0.568339 3.14159" />
+			<geometry>
+				<mesh filename="file://$(find al5d_description)/urdf/al5d/asb-04.stl"/>
+			</geometry>
+			<material name="asb-04_material">
+				<color rgba="0.647059 0.647059 0.647059 1.0"/>
+			</material>
+		</collision>
+		<collision>
+			<origin xyz="-0.168036 -0.0235167 0.101822" rpy="-1.5708 -1.00246 8.92593e-15" />
+			<geometry>
+				<mesh filename="file://$(find al5d_description)/urdf/al5d/imported10.stl"/>
+			</geometry>
+			<material name="imported10_material">
+				<color rgba="0.972549 0.529412 0.00392157 1.0"/>
+			</material>
+		</collision>
+		<collision>
+			<origin xyz="-0.031327 -0.0220573 0.0216741" rpy="0.568339 3.54935e-15 1.5708" />
+			<geometry>
+				<mesh filename="file://$(find al5d_description)/urdf/al5d/hub-08.stl"/>
+			</geometry>
+			<material name="hub-08_material">
+				<color rgba="0.917647 0.917647 0.917647 1.0"/>
+			</material>
+		</collision>
+		<visual>
+			<origin xyz="0 0 0" rpy="0 -0 0" />
+			<geometry>
+				<mesh filename="file://$(find al5d_description)/urdf/al5d/elbow_1.stl"/>
+			</geometry>
+			<material name="elbow_1_material">
+				<color rgba="0.821471 0.601159 0.31861 1.0"/>
+			</material>
+		</visual>
+		<inertial>
+			<origin xyz="-0.12068 -0.022989 0.0749584" rpy="0 0 0"/>
+			<mass value="1.12468" />
+			<inertia ixx="0.00239634" ixy="4.82258e-05"  ixz="0.00330002" iyy="0.00794344" iyz="2.52644e-05" izz="0.00587491" />
+		</inertial>
+	</link>
+	<link name="arm_1">
+		<collision>
+			<origin xyz="-3.38618e-15 -0.0297627 -0.0823056" rpy="4.45083e-16 -1.30243e-15 -3.14159" />
 			<geometry>
 				<mesh filename="file://$(find al5d_description)/urdf/al5d/imported6.stl"/>
@@ -13,14 +189,5 @@
 		</collision>
 		<collision>
-			<origin xyz="-0.0644966 -0.0884144 0.0797579" rpy="-1.24918 0.0119563 -1.42627" />
-			<geometry>
-				<mesh filename="file://$(find al5d_description)/urdf/al5d/imported4.stl"/>
-			</geometry>
-			<material name="imported4_material">
-				<color rgba="0.231373 0.380392 0.705882 1.0"/>
-			</material>
-		</collision>
-		<collision>
-			<origin xyz="-0.0749532 -0.0165706 0.0806259" rpy="-1.24918 0.0119563 -1.42627" />
+			<origin xyz="0.000965268 -0.0599498 -0.000537904" rpy="-0.496906 9.71233e-16 -1.5708" />
 			<geometry>
 				<mesh filename="file://$(find al5d_description)/urdf/al5d/imported5.stl"/>
@@ -31,5 +198,14 @@
 		</collision>
 		<collision>
-			<origin xyz="0.064324 -0.00303524 0.126312" rpy="-2.68503 -0.0119563 1.71533" />
+			<origin xyz="-3.71925e-15 0.0070373 -0.146277" rpy="9.96212e-16 3.55487e-16 1.5708" />
+			<geometry>
+				<mesh filename="file://$(find al5d_description)/urdf/al5d/imported4.stl"/>
+			</geometry>
+			<material name="imported4_material">
+				<color rgba="0.231373 0.380392 0.705882 1.0"/>
+			</material>
+		</collision>
+		<collision>
+			<origin xyz="-3.64986e-15 -0.0655687 -0.146277" rpy="1.11629e-15 3.24625e-16 1.5708" />
 			<geometry>
 				<mesh filename="file://$(find al5d_description)/urdf/al5d/imported5.stl"/>
@@ -40,5 +216,5 @@
 		</collision>
 		<collision>
-			<origin xyz="-0.00195659 -0.00857929 0.0920755" rpy="1.53299 -1.24896 -2.96119" />
+			<origin xyz="-0.0123063 -0.0631002 -0.073025" rpy="1.5708 8.15346e-16 3.44632e-16" />
 			<geometry>
 				<mesh filename="file://$(find al5d_description)/urdf/al5d/asb203.stl"/>
@@ -49,5 +225,5 @@
 		</collision>
 		<collision>
-			<origin xyz="0.0721877 -0.0639893 0.126053" rpy="-0.037808 -1.24896 -2.96119" />
+			<origin xyz="1.38778e-17 0.002 -2.77556e-17" rpy="1.95874e-19 4.38707e-17 -8.6926e-19" />
 			<geometry>
 				<mesh filename="file://$(find al5d_description)/urdf/al5d/imported8.stl"/>
@@ -60,19 +236,37 @@
 			<origin xyz="0 0 0" rpy="0 -0 0" />
 			<geometry>
-				<mesh filename="file://$(find al5d_description)/urdf/al5d/assembly_3_1.stl"/>
-			</geometry>
-			<material name="assembly_3_1_material">
+				<mesh filename="file://$(find al5d_description)/urdf/al5d/arm_1.stl"/>
+			</geometry>
+			<material name="arm_1_material">
 				<color rgba="0.549634 0.627756 0.687007 1.0"/>
 			</material>
 		</visual>
 		<inertial>
-			<origin xyz="-0.0150037 -0.0519635 0.098131" rpy="0 0 0"/>
+			<origin xyz="4.99624e-05 -0.0221487 -0.0892021" rpy="0 0 0"/>
 			<mass value="0.210521" />
-			<inertia ixx="0.000316475" ixy="-0.000161476"  ixz="-0.000134923" iyy="0.000638896" iyz="-6.90695e-05" izz="0.000738837" />
-		</inertial>
-	</link>
-	<link name="assembly_6_1">
-		<collision>
-			<origin xyz="0.014478 -0.014986 -0.061214" rpy="-1.01359e-18 4.12165e-17 -2.99908e-19" />
+			<inertia ixx="0.000832208" ixy="3.97597e-07"  ixz="-9.32581e-07" iyy="0.000627814" iyz="0.000105361" izz="0.000229822" />
+		</inertial>
+	</link>
+	<link name="shoulder_1">
+		<collision>
+			<origin xyz="0.02269 -0.00174611 -0.036506" rpy="1.5708 -1.5708 0" />
+			<geometry>
+				<mesh filename="file://$(find al5d_description)/urdf/al5d/imported2.stl"/>
+			</geometry>
+			<material name="imported2_material">
+				<color rgba="0.768627 0.886275 0.952941 1.0"/>
+			</material>
+		</collision>
+		<collision>
+			<origin xyz="-0.0118691 0.07126 -0.0250047" rpy="-3.14159 -1.5708 0" />
+			<geometry>
+				<mesh filename="file://$(find al5d_description)/urdf/al5d/imported1.stl"/>
+			</geometry>
+			<material name="imported1_material">
+				<color rgba="0.972549 0.529412 0.00392157 1.0"/>
+			</material>
+		</collision>
+		<collision>
+			<origin xyz="0.014478 -0.014986 -0.061214" rpy="4.38009e-20 9.13044e-19 1.68915e-18" />
 			<geometry>
 				<mesh filename="file://$(find al5d_description)/urdf/al5d/hs-805bb.stl"/>
@@ -82,28 +276,10 @@
 			</material>
 		</collision>
-		<collision>
-			<origin xyz="0.02269 -0.00174611 -0.036506" rpy="1.5708 -1.5708 0" />
-			<geometry>
-				<mesh filename="file://$(find al5d_description)/urdf/al5d/imported2.stl"/>
-			</geometry>
-			<material name="imported2_material">
-				<color rgba="0.768627 0.886275 0.952941 1.0"/>
-			</material>
-		</collision>
-		<collision>
-			<origin xyz="-0.0118691 0.07126 -0.0250047" rpy="-3.14159 -1.5708 0" />
-			<geometry>
-				<mesh filename="file://$(find al5d_description)/urdf/al5d/imported1.stl"/>
-			</geometry>
-			<material name="imported1_material">
-				<color rgba="0.972549 0.529412 0.00392157 1.0"/>
-			</material>
-		</collision>
-		<visual>
-			<origin xyz="0 0 0" rpy="0 -0 0" />
-			<geometry>
-				<mesh filename="file://$(find al5d_description)/urdf/al5d/assembly_6_1.stl"/>
-			</geometry>
-			<material name="assembly_6_1_material">
+		<visual>
+			<origin xyz="0 0 0" rpy="0 -0 0" />
+			<geometry>
+				<mesh filename="file://$(find al5d_description)/urdf/al5d/shoulder_1.stl"/>
+			</geometry>
+			<material name="shoulder_1_material">
 				<color rgba="0.908985 0.833727 0.73777 1.0"/>
 			</material>
@@ -115,25 +291,25 @@
 		</inertial>
 	</link>
-	<link name="assembly_1_1">
-		<collision>
-			<origin xyz="-0.0417983 -0.04424 0.0695052" rpy="-1.5708 1.49702e-19 2.03954e-20" />
-			<geometry>
-				<mesh filename="file://$(find al5d_description)/urdf/al5d/servomotore_hitec_hs485-hb.stl"/>
-			</geometry>
-			<material name="servomotore_hitec_hs485-hb_material">
-				<color rgba="0.792157 0.819608 0.933333 1.0"/>
-			</material>
-		</collision>
-		<collision>
-			<origin xyz="-0.0417983 -0.04424 0.0695052" rpy="-1.5708 1.49702e-19 2.03954e-20" />
-			<geometry>
-				<mesh filename="file://$(find al5d_description)/urdf/al5d/part_3.stl"/>
-			</geometry>
-			<material name="part_3_material">
-				<color rgba="0.792157 0.819608 0.933333 1.0"/>
-			</material>
-		</collision>
-		<collision>
-			<origin xyz="-3.53884e-16 -0.0465764 -3.60822e-16" rpy="3.14159 3.16747e-17 -3.14159" />
+	<link name="base_1">
+		<collision>
+			<origin xyz="1.38778e-17 -0.0408164 0" rpy="-1.5708 -3.71498e-17 -8.77933e-18" />
+			<geometry>
+				<mesh filename="file://$(find al5d_description)/urdf/al5d/imported36.stl"/>
+			</geometry>
+			<material name="imported36_material">
+				<color rgba="0.917647 0.917647 0.917647 1.0"/>
+			</material>
+		</collision>
+		<collision>
+			<origin xyz="0.0565 -0.0408164 3.46945e-18" rpy="-1.5708 -3.72385e-17 -1.22544e-17" />
+			<geometry>
+				<mesh filename="file://$(find al5d_description)/urdf/al5d/imported36.stl"/>
+			</geometry>
+			<material name="imported36_material">
+				<color rgba="0.917647 0.917647 0.917647 1.0"/>
+			</material>
+		</collision>
+		<collision>
+			<origin xyz="0 -0.0423164 3.46945e-18" rpy="1.51444e-18 2.5486e-19 -1.00323e-19" />
 			<geometry>
 				<mesh filename="file://$(find al5d_description)/urdf/al5d/imported1.stl"/>
@@ -143,250 +319,72 @@
 			</material>
 		</collision>
-		<collision>
-			<origin xyz="-3.46945e-16 -0.0480764 -3.747e-16" rpy="-1.5708 -3.15605e-16 1.67908e-15" />
-			<geometry>
-				<mesh filename="file://$(find al5d_description)/urdf/al5d/imported36.stl"/>
-			</geometry>
-			<material name="imported36_material">
-				<color rgba="0.917647 0.917647 0.917647 1.0"/>
-			</material>
-		</collision>
-		<collision>
-			<origin xyz="-0.0417983 -0.04424 0.0695052" rpy="-1.5708 1.49702e-19 2.03954e-20" />
-			<geometry>
-				<mesh filename="file://$(find al5d_description)/urdf/al5d/part_5.stl"/>
-			</geometry>
-			<material name="part_5_material">
-				<color rgba="0.792157 0.819608 0.933333 1.0"/>
-			</material>
-		</collision>
-		<collision>
-			<origin xyz="-0.0417983 -0.04424 0.0695052" rpy="-1.5708 1.49702e-19 2.03954e-20" />
-			<geometry>
-				<mesh filename="file://$(find al5d_description)/urdf/al5d/part_4.stl"/>
-			</geometry>
-			<material name="part_4_material">
-				<color rgba="0.792157 0.819608 0.933333 1.0"/>
-			</material>
-		</collision>
-		<collision>
-			<origin xyz="0 -0.0065 6.93889e-18" rpy="2.67186e-19 1.49702e-19 2.03954e-20" />
-			<geometry>
-				<mesh filename="file://$(find al5d_description)/urdf/al5d/ingranaggio_dentato_innesto_servomotore.stl"/>
-			</geometry>
-			<material name="ingranaggio_dentato_innesto_servomotore_material">
-				<color rgba="0.792157 0.819608 0.933333 1.0"/>
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