Commit message: Add files via upload

File: al5d/al5d_description/urdf/al5d/robot.urdf (robot description, URDF)
Before this commit: robot onshape, 7 links, 6 joints
Links:
- removed link assembly_10_1
- removed link assembly_11_1
- removed link assembly_1_1
- removed link assembly_3_1
- removed link assembly_4_1
- removed link assembly_5_1
- removed link assembly_6_1
- added link arm_1, mass 0.210521; collision mesh filename=package://asb203.stl; collision mesh filename=package://imported4.stl
- added link base_1, mass 0.859229; collision mesh filename=package://imported1.stl; collision mesh filename=package://imported36.stl
- added link elbow_1, mass 1.12468; collision mesh filename=package://asb-04.stl; collision mesh filename=package://asb201b.stl
- added link gripper1_1, mass 0.00484154; collision mesh filename=package://gripper_finger_pad.stl; collision mesh filename=package://gripper_finger_right.stl
- added link gripper2_1, mass 0.00484161; collision mesh filename=package://gripper_finger_left.stl; collision mesh filename=package://gripper_finger_pad.stl
- added link hand_1, mass 0.237212; collision mesh filename=package://gripper_wrist.stl; collision mesh filename=package://horn.stl
- added link shoulder_1, mass 1.2783; collision mesh filename=package://hs-805bb.stl; collision mesh filename=package://imported1.stl
- added link wrist_1, mass 0.0622741; collision mesh filename=package://bb-03.stl; collision mesh filename=package://imported15.stl
Joints:
- removed joint 1
- removed joint 2
- removed joint 3
- removed joint 4
- removed joint 5
- removed joint 6
- added joint joint1: type revolute, parent shoulder_1, child base_1, origin xyz=-0.0118691 0.030112 -0.0250047 rpy=3.14159 1.5708 0, axis 0 1 0, limit lower=0 upper=6.28319 effort=1 velocity=20
- added joint joint2: type revolute, parent arm_1, child shoulder_1, origin xyz=-3.55271e-15 0.0004373 -0.146277 rpy=-1.5708 0.877711 5.8629e-15, axis 0 0 1, limit lower=-1.5708 upper=2.0944 effort=1 velocity=20
- added joint joint3: type revolute, parent elbow_1, child arm_1, origin xyz=-0.153811 0.00723332 0.092738 rpy=-3.14159 -0.0714328 3.14159, axis 0 -1 0, limit lower=-2.35619 upper=2.35619 effort=1 velocity=20
- added joint joint4: type revolute, parent wrist_1, child elbow_1, origin xyz=-0.0599957 -0.29722 0.125782 rpy=-3.13392 0.961817 -1.55889, axis 0 -1 0, limit lower=-2.53073 upper=2.53073 effort=1 velocity=20
- added joint joint5: type revolute, parent wrist_1, child hand_1, origin xyz=-0.0290255 -0.329587 0.0791964 rpy=-0.00535255 0.608959 1.57334, axis 0 0 1, limit lower=0 upper=6.28319 effort=1 velocity=20
- added joint joint6: type prismatic, parent hand_1, child gripper1_1, origin xyz=0.0194818 -3.46945e-18 -0.0280252 rpy=-2.08852e-16 1.5708 0, axis 0 0 -1, limit lower=0.0005 upper=0.0012 effort=1 velocity=20
- added joint joint7: type prismatic, parent hand_1, child gripper2_1, origin xyz=-0.0017018 3.46945e-18 -0.0280252 rpy=3.14159 1.5708 0, axis 0 0 -1, limit lower=0.0005 upper=0.0012 effort=1 velocity=20
